Commit message: Add Mecanum drive plugin for Gazebo simulation
- Created MecanumCmd.msg for command messages with velocity and rotation.
- Added package.xml for the mecanum_gazebo_plugin with dependencies.
- Implemented plugin_description.xml for the MecanumDrivePlugin.
- Developed mecanum_drive_plugin.cpp to control the robot's movement using ROS messages.
- Integrated joint control for the four wheels based on received commands.

File: MY-Robot/urdf/MY-Robot.urdf (robot description, URDF)
Before this commit: robot MY-Robot, 7 links, 6 joints
Links:
- removed link base_footprint
Joints:
- removed joint base_joint

File: chassis/install/chassis/share/chassis/urdf/chassis.xacro (robot description, xacro)
@@ -5,31 +5,21 @@
 <robot name="chassis" xmlns:xacro="http://www.ros.org/wiki/xacro">
   <!-- ========== 仿真/实物切换参数 ========== -->
+  <xacro:include filename="$(find chassis)/urdf/scan_sensor.xacro" />
   <xacro:arg name="use_sim" default="true"/>
-  <xacro:arg name="control_yaml" default="$(find chassis)/config/chassis_control.yaml"/>
-  <!-- 引入宏定义文件 -->
-  <xacro:include filename="$(find chassis)/urdf/scan_sensor.xacro" />
-  <xacro:include filename="$(find chassis)/urdf/gazebo_mecanum.xacro" />
-  <!-- 虚拟根坐标系（地面投影） -->
-  <link name="base_footprint"/>
-  <joint name="base_joint" type="fixed">
-    <parent link="base_footprint"/>
-    <child link="base_link"/>
-    <origin xyz="0 0 0.078" rpy="0 0 0"/>   <!-- 提升底盘 -->
-  </joint>
   <link
     name="base_link">
     <inertial>
       <origin
-        xyz="-0.0677269794437447 4.32361658823655E-05 0.0669607519587934"
-        rpy="0 0 0" />
-      <mass
-        value="3.25970439008785" />
-      <inertia
-        ixx="0.0187796297594545"
-        ixy="-4.77646510491924E-08"
-        ixz="1.83706592921599E-09"
-        iyy="0.0204875409369385"
-        iyz="3.19329644861363E-08"
-        izz="0.0375114470548974" />
+        xyz="-0.0677499107956596 4.3724418912483E-05 0.0683926250538354"
+        rpy="0 0 0" />
+      <mass
+        value="3.22393142364253" />
+      <inertia
+        ixx="0.0187770652552285"
+        ixy="-6.94989088987062E-08"
+        ixz="-3.69535574562707E-08"
+        iyy="0.02048392582904"
+        iyz="3.35166257416731E-11"
+        izz="0.0375088689683629" />
     </inertial>
     <visual>
@@ -61,15 +51,15 @@
     <inertial>
       <origin
-        xyz="-0.00250631530381207 4.56584853764097E-06 0.00608264669062358"
-        rpy="0 0 0" />
-      <mass
-        value="0.0374307357500632" />
-      <inertia
-        ixx="2.80476493090254E-05"
-        ixy="-2.19899695279442E-09"
-        ixz="-1.07121854785563E-06"
-        iyy="3.36164872297249E-05"
-        iyz="-6.83968851717712E-10"
-        izz="4.50845442757731E-05" />
+        xyz="-0.0025063 4.5658E-06 0.0060826"
+        rpy="0 0 0" />
+      <mass
+        value="0.037431" />
+      <inertia
+        ixx="2.8048E-05"
+        ixy="-2.199E-09"
+        ixz="-1.0712E-06"
+        iyy="3.3616E-05"
+        iyz="-6.8397E-10"
+        izz="4.5085E-05" />
     </inertial>
     <visual>
@@ -84,5 +74,5 @@
         name="">
         <color
-          rgba="0.376470588235294 0.376470588235294 0.376470588235294 1" />
+          rgba="0.37647 0.37647 0.37647 1" />
       </material>
     </visual>
@@ -114,15 +104,15 @@
     <inertial>
       <origin
-        xyz="-1.40050867430963E-08 -0.0140076625586234 2.61687240835085E-08"
-        rpy="0 0 0" />
-      <mass
-        value="0.0481550141943844" />
-      <inertia
-        ixx="2.03928872568603E-05"
-        ixy="-4.78408666290658E-12"
-        ixz="-8.22422789230428E-12"
-        iyy="3.30574790370537E-05"
-        iyz="2.64993040628741E-12"
-        izz="2.03928695670075E-05" />
+        xyz="-2.268E-05 -0.017766 -3.3245E-05"
+        rpy="0 0 0" />
+      <mass
+        value="0.057098" />
+      <inertia
+        ixx="2.1034E-05"
+        ixy="5.4288E-09"
+        ixz="9.6894E-09"
+        iyy="3.3961E-05"
+        iyz="7.9775E-09"
+        izz="2.1037E-05" />
     </inertial>
     <visual>
@@ -137,5 +127,5 @@
         name="">
         <color
-          rgba="0.792156862745098 0.819607843137255 0.933333333333333 1" />
+          rgba="0.79216 0.81961 0.93333 1" />
       </material>
     </visual>
@@ -167,15 +157,15 @@
     <inertial>
       <origin
-        xyz="-1.40050869512631E-08 0.0139923374413648 2.61687235492136E-08"
-        rpy="0 0 0" />
-      <mass
-        value="0.0481550141943843" />
-      <inertia
-        ixx="2.03928872568601E-05"
-        ixy="-4.78408655172236E-12"
-        ixz="-8.22422789557072E-12"
-        iyy="3.30574790370536E-05"
-        iyz="2.64993057879603E-12"
-        izz="2.03928695670075E-05" />
+        xyz="-2.268E-05 0.017753 -3.3245E-05"
+        rpy="0 0 0" />
+      <mass
+        value="0.057098" />
+      <inertia
+        ixx="2.1034E-05"
+        ixy="5.4288E-09"
+        ixz="9.6894E-09"
+        iyy="3.3961E-05"
+        iyz="7.9775E-09"
+        izz="2.1037E-05" />
     </inertial>
     <visual>
@@ -190,5 +180,5 @@
         name="">
         <color
-          rgba="0.792156862745098 0.819607843137255 0.933333333333333 1" />
+          rgba="0.79216 0.81961 0.93333 1" />
       </material>
     </visual>
@@ -220,15 +210,15 @@
     <inertial>
       <origin
-        xyz="-1.40050894978372E-08 -0.0140076625586241 2.61687244512698E-08"
-        rpy="0 0 0" />
-      <mass
-        value="0.0481550141943849" />
-      <inertia
-        ixx="2.03928872568603E-05"
-        ixy="-4.78408662746301E-12"
-        ixz="-8.22422788926722E-12"
-        iyy="3.3057479037054E-05"
-        iyz="2.64993046458594E-12"
-        izz="2.03928695670077E-05" />
+        xyz="-2.268E-05 -0.017766 -3.3245E-05"
+        rpy="0 0 0" />
+      <mass
+        value="0.057098" />
+      <inertia
+        ixx="2.1034E-05"
+        ixy="5.4288E-09"
+        ixz="9.6894E-09"
+        iyy="3.3961E-05"
+        iyz="7.9775E-09"
+        izz="2.1037E-05" />
     </inertial>
     <visual>
@@ -243,5 +233,5 @@
         name="">
         <color
-          rgba="0.792156862745098 0.819607843137255 0.933333333333333 1" />
+          rgba="0.79216 0.81961 0.93333 1" />
       </material>
     </visual>
@@ -273,15 +263,15 @@
     <inertial>
       <origin
-        xyz="-1.40050829475213E-08 0.0139923374413657 2.61687230843077E-08"
-        rpy="0 0 0" />
-      <mass
-        value="0.0481550141943844" />
-      <inertia
-        ixx="2.03928872568602E-05"
-        ixy="-4.7840865501743E-12"
-        ixz="-8.22422789329745E-12"
-        iyy="3.30574790370536E-05"
-        iyz="2.64993059290757E-12"
-        izz="2.03928695670075E-05" />
+        xyz="-2.268E-05 0.017753 -3.3245E-05"
+        rpy="0 0 0" />
+      <mass
+        value="0.057098" />
+      <inertia
+        ixx="2.1034E-05"
+        ixy="5.4288E-09"
+        ixz="9.6894E-09"
+        iyy="3.3961E-05"
+        iyz="7.9775E-09"
+        izz="2.1037E-05" />
     </inertial>
     <visual>
@@ -296,5 +286,5 @@
         name="">
         <color
-          rgba="0.792156862745098 0.819607843137255 0.933333333333333 1" />
+          rgba="0.79216 0.81961 0.93333 1" />
       </material>
     </visual>
@@ -322,6 +312,51 @@
       xyz="0 1 0" />
   </joint>
-  <!-- 调用宏，生成传感器和驱动 -->
+  <gazebo reference="FL_Link">
+    <mu1>100.0</mu1>
+    <mu2>100.0</mu2>
+    <kp>100000000.0</kp>
+    <kd>10.0</kd>
+  </gazebo>
+  <gazebo reference="FR_Link">
+    <mu1>100.0</mu1>
+    <mu2>100.0</mu2>
+    <kp>100000000.0</kp>
+    <kd>10.0</kd>
+  </gazebo>
+  <gazebo reference="BL_Link">
+    <mu1>100.0</mu1>
+    <mu2>100.0</mu2>
+    <kp>100000000.0</kp>
+    <kd>10.0</kd>
+  </gazebo>
+  <gazebo reference="BR_Link">
+    <mu1>100.0</mu1>
+    <mu2>100.0</mu2>
+    <kp>100000000.0</kp>
+    <kd>10.0</kd>
+  </gazebo>
+  <gazebo>
+    <plugin name="my_mecanum_plugin" filename="libmecanum_drive_plugin.so">
+      <fl_joint>FL_Joint</fl_joint>
+      <fr_joint>FR_Joint</fr_joint>
+      <bl_joint>BL_Joint</bl_joint>
+      <br_joint>BR_Joint</br_joint>
+      <wheel_radius>0.0375</wheel_radius>
+      <wheel_base>0.1550</wheel_base>
+      <track_width>0.4166</track_width>
+    </plugin>
+  </gazebo>
+  <gazebo>
+    <plugin name="joint_state_publisher" filename="libgazebo_ros_joint_state_publisher.so">
+      <ros>
+        <remapping>~/out:=joint_states</remapping>
+      </ros>
+      <update_rate>50</update_rate>
+      <joint_name>FL_Joint</joint_name>
+      <joint_name>FR_Joint</joint_name>
+      <joint_name>BL_Joint</joint_name>
+      <joint_name>BR_Joint</joint_name>
+    </plugin>
+  </gazebo>
   <xacro:scan_sensor prefix="scan" use_sim="$(arg use_sim)"/>
-  <xacro:mecanum_drive use_sim="$(arg use_sim)"/>
 </robot>

File: chassis/install/chassis/share/chassis/urdf/gazebo_mecanum.xacro (robot description, xacro)
@@ -3,36 +3,33 @@
   <xacro:macro name="mecanum_drive" params="use_sim:=true">
     <xacro:if value="${use_sim}">
-      <!-- 加载 gazebo_ros2_control 插件 -->
       <gazebo>
-        <plugin name="gazebo_ros2_control" filename="libgazebo_ros2_control.so">
-          <parameters>$(find chassis)/config/chassis_control.yaml</parameters>
+        <plugin name="mecanum_drive" filename="libgazebo_ros_mecanum_drive.so">
+          <ros>
+            <remapping>cmd_vel:=cmd_vel</remapping>
+          </ros>
+          <left_front_joint>FL_Joint</left_front_joint>
+          <right_front_joint>FR_Joint</right_front_joint>
+          <left_rear_joint>BL_Joint</left_rear_joint>
+          <right_rear_joint>BR_Joint</right_rear_joint>
+          <wheel_radius>0.0375</wheel_radius>
+          <wheel_separation>0.4166</wheel_separation>
+          <wheel_base>0.1550</wheel_base>
+          <robot_base_frame>base_link</robot_base_frame>
+          <odometry_frame>odom</odometry_frame>
+          <publish_wheel_tf>false</publish_wheel_tf>
+          <publish_odometry>true</publish_odometry>
+          <publish_odom_tf>true</publish_odom_tf>
+        </plugin>
+        <plugin name="joint_state_publisher" filename="libgazebo_ros_joint_state_publisher.so">
+          <ros>
+            <remapping>~/out:=joint_states</remapping>
+          </ros>
+          <update_rate>30</update_rate>
+          <joint_name>FL_Joint</joint_name>
+          <joint_name>FR_Joint</joint_name>
+          <joint_name>BL_Joint</joint_name>
+          <joint_name>BR_Joint</joint_name>
         </plugin>
       </gazebo>
-      <!-- 定义硬件接口（ros2_control 必须） -->
-      <ros2_control name="GazeboSystem" type="system">
-        <hardware>
-          <plugin>gazebo_ros2_control/GazeboSystem</plugin>
-        </hardware>
-        <joint name="FL_Joint">
-          <command_interface name="velocity"/>
-          <state_interface name="position"/>
-          <state_interface name="velocity"/>
-        </joint>
-        <joint name="FR_Joint">
-          <command_interface name="velocity"/>
-          <state_interface name="position"/>
-          <state_interface name="velocity"/>
-        </joint>
-        <joint name="BL_Joint">
-          <command_interface name="velocity"/>
-          <state_interface name="position"/>
-          <state_interface name="velocity"/>
-        </joint>
-        <joint name="BR_Joint">
-          <command_interface name="velocity"/>
-          <state_interface name="position"/>
-          <state_interface name="velocity"/>
-        </joint>
-      </ros2_control>
     </xacro:if>
   </xacro:macro>

File: chassis/urdf/chassis.urdf (robot description, URDF)
Before this commit: robot chassis, 6 links, 5 joints
Links:
- link BL_Link: mass 0.0481550141943849 -> 0.057098
- link BR_Link: mass 0.0481550141943844 -> 0.057098
- link FL_Link: mass 0.0481550141943844 -> 0.057098
- link FR_Link: mass 0.0481550141943843 -> 0.057098
- link base_link: mass 3.25970439008785 -> 3.22393142364253
- link scan_Link: mass 0.0374307357500632 -> 0.037431

File: chassis/urdf/chassis.xacro (robot description, xacro)
@@ -5,31 +5,21 @@
 <robot name="chassis" xmlns:xacro="http://www.ros.org/wiki/xacro">
   <!-- ========== 仿真/实物切换参数 ========== -->
+  <xacro:include filename="$(find chassis)/urdf/scan_sensor.xacro" />
   <xacro:arg name="use_sim" default="true"/>
-  <xacro:arg name="control_yaml" default="$(find chassis)/config/chassis_control.yaml"/>
-  <!-- 引入宏定义文件 -->
-  <xacro:include filename="$(find chassis)/urdf/scan_sensor.xacro" />
-  <xacro:include filename="$(find chassis)/urdf/gazebo_mecanum.xacro" />
-  <!-- 虚拟根坐标系（地面投影） -->
-  <link name="base_footprint"/>
-  <joint name="base_joint" type="fixed">
-    <parent link="base_footprint"/>
-    <child link="base_link"/>
-    <origin xyz="0 0 0.078" rpy="0 0 0"/>   <!-- 提升底盘 -->
-  </joint>
   <link
     name="base_link">
     <inertial>
       <origin
-        xyz="-0.0677269794437447 4.32361658823655E-05 0.0669607519587934"
-        rpy="0 0 0" />
-      <mass
-        value="3.25970439008785" />
-      <inertia
-        ixx="0.0187796297594545"
-        ixy="-4.77646510491924E-08"
-        ixz="1.83706592921599E-09"
-        iyy="0.0204875409369385"
-        iyz="3.19329644861363E-08"
-        izz="0.0375114470548974" />
+        xyz="-0.0677499107956596 4.3724418912483E-05 0.0683926250538354"
+        rpy="0 0 0" />
+      <mass
+        value="3.22393142364253" />
+      <inertia
+        ixx="0.0187770652552285"
+        ixy="-6.94989088987062E-08"
+        ixz="-3.69535574562707E-08"
+        iyy="0.02048392582904"
+        iyz="3.35166257416731E-11"
+        izz="0.0375088689683629" />
     </inertial>
     <visual>
@@ -61,15 +51,15 @@
     <inertial>
       <origin
-        xyz="-0.00250631530381207 4.56584853764097E-06 0.00608264669062358"
-        rpy="0 0 0" />
-      <mass
-        value="0.0374307357500632" />
-      <inertia
-        ixx="2.80476493090254E-05"
-        ixy="-2.19899695279442E-09"
-        ixz="-1.07121854785563E-06"
-        iyy="3.36164872297249E-05"
-        iyz="-6.83968851717712E-10"
-        izz="4.50845442757731E-05" />
+        xyz="-0.0025063 4.5658E-06 0.0060826"
+        rpy="0 0 0" />
+      <mass
+        value="0.037431" />
+      <inertia
+        ixx="2.8048E-05"
+        ixy="-2.199E-09"
+        ixz="-1.0712E-06"
+        iyy="3.3616E-05"
+        iyz="-6.8397E-10"
+        izz="4.5085E-05" />
     </inertial>
     <visual>
@@ -84,5 +74,5 @@
         name="">
         <color
-          rgba="0.376470588235294 0.376470588235294 0.376470588235294 1" />
+          rgba="0.37647 0.37647 0.37647 1" />
       </material>
     </visual>
@@ -114,15 +104,15 @@
     <inertial>
       <origin
-        xyz="-1.40050867430963E-08 -0.0140076625586234 2.61687240835085E-08"
-        rpy="0 0 0" />
-      <mass
-        value="0.0481550141943844" />
-      <inertia
-        ixx="2.03928872568603E-05"
-        ixy="-4.78408666290658E-12"
-        ixz="-8.22422789230428E-12"
-        iyy="3.30574790370537E-05"
-        iyz="2.64993040628741E-12"
-        izz="2.03928695670075E-05" />
+        xyz="-2.268E-05 -0.017766 -3.3245E-05"
+        rpy="0 0 0" />
+      <mass
+        value="0.057098" />
+      <inertia
+        ixx="2.1034E-05"
+        ixy="5.4288E-09"
+        ixz="9.6894E-09"
+        iyy="3.3961E-05"
+        iyz="7.9775E-09"
+        izz="2.1037E-05" />
     </inertial>
     <visual>
@@ -137,5 +127,5 @@
         name="">
         <color
-          rgba="0.792156862745098 0.819607843137255 0.933333333333333 1" />
+          rgba="0.79216 0.81961 0.93333 1" />
       </material>
     </visual>
@@ -167,15 +157,15 @@
     <inertial>
       <origin
-        xyz="-1.40050869512631E-08 0.0139923374413648 2.61687235492136E-08"
-        rpy="0 0 0" />
-      <mass
-        value="0.0481550141943843" />
-      <inertia
-        ixx="2.03928872568601E-05"
-        ixy="-4.78408655172236E-12"
-        ixz="-8.22422789557072E-12"
-        iyy="3.30574790370536E-05"
-        iyz="2.64993057879603E-12"
-        izz="2.03928695670075E-05" />
+        xyz="-2.268E-05 0.017753 -3.3245E-05"
+        rpy="0 0 0" />
+      <mass
+        value="0.057098" />
+      <inertia
+        ixx="2.1034E-05"
+        ixy="5.4288E-09"
+        ixz="9.6894E-09"
+        iyy="3.3961E-05"
+        iyz="7.9775E-09"
+        izz="2.1037E-05" />
     </inertial>
     <visual>
@@ -190,5 +180,5 @@
         name="">
         <color
-          rgba="0.792156862745098 0.819607843137255 0.933333333333333 1" />
+          rgba="0.79216 0.81961 0.93333 1" />
       </material>
     </visual>
@@ -220,15 +210,15 @@
     <inertial>
       <origin
-        xyz="-1.40050894978372E-08 -0.0140076625586241 2.61687244512698E-08"
-        rpy="0 0 0" />
-      <mass
-        value="0.0481550141943849" />
-      <inertia
-        ixx="2.03928872568603E-05"
-        ixy="-4.78408662746301E-12"
-        ixz="-8.22422788926722E-12"
-        iyy="3.3057479037054E-05"
-        iyz="2.64993046458594E-12"
-        izz="2.03928695670077E-05" />
+        xyz="-2.268E-05 -0.017766 -3.3245E-05"
+        rpy="0 0 0" />
+      <mass
+        value="0.057098" />
+      <inertia
+        ixx="2.1034E-05"
+        ixy="5.4288E-09"
+        ixz="9.6894E-09"
+        iyy="3.3961E-05"
+        iyz="7.9775E-09"
+        izz="2.1037E-05" />
     </inertial>
     <visual>
@@ -243,5 +233,5 @@
         name="">
         <color
-          rgba="0.792156862745098 0.819607843137255 0.933333333333333 1" />
+          rgba="0.79216 0.81961 0.93333 1" />
       </material>
     </visual>
@@ -273,15 +263,15 @@
     <inertial>
       <origin
-        xyz="-1.40050829475213E-08 0.0139923374413657 2.61687230843077E-08"
-        rpy="0 0 0" />
-      <mass
-        value="0.0481550141943844" />
-      <inertia
-        ixx="2.03928872568602E-05"
-        ixy="-4.7840865501743E-12"
-        ixz="-8.22422789329745E-12"
-        iyy="3.30574790370536E-05"
-        iyz="2.64993059290757E-12"
-        izz="2.03928695670075E-05" />
+        xyz="-2.268E-05 0.017753 -3.3245E-05"
+        rpy="0 0 0" />
+      <mass
+        value="0.057098" />
+      <inertia
+        ixx="2.1034E-05"
+        ixy="5.4288E-09"
+        ixz="9.6894E-09"
+        iyy="3.3961E-05"
+        iyz="7.9775E-09"
+        izz="2.1037E-05" />
     </inertial>
     <visual>
@@ -296,5 +286,5 @@
         name="">
         <color
-          rgba="0.792156862745098 0.819607843137255 0.933333333333333 1" />
+          rgba="0.79216 0.81961 0.93333 1" />
       </material>
     </visual>
@@ -322,6 +312,4 @@
       xyz="0 1 0" />
   </joint>
-  <!-- 调用宏，生成传感器和驱动 -->
   <xacro:scan_sensor prefix="scan" use_sim="$(arg use_sim)"/>
-  <xacro:mecanum_drive use_sim="$(arg use_sim)"/>
 </robot>
