Commit message: Add UnifiedOdometry node for simulating odometry calculations
- Implemented a new ROS2 node that calculates odometry based on joint states.
- Supports both simulation and real robot modes (real mode not fully implemented).
- Publishes odometry data and transforms using TF2.
- Parameters for wheel radius, wheel base, track width, and frames are configurable via ROS parameters.

File: chassis/install/chassis/share/chassis/urdf/chassis.xacro (robot description, xacro)
@@ -5,6 +5,10 @@
 <robot name="chassis" xmlns:xacro="http://www.ros.org/wiki/xacro">
   <!-- ========== 仿真/实物切换参数 ========== -->
+  <xacro:arg name="use_sim" default="true"/>
+  <xacro:property name="mecanum_config" value="$(find chassis)/config/robot_config.yaml" />
   <xacro:include filename="$(find chassis)/urdf/scan_sensor.xacro" />
-  <xacro:arg name="use_sim" default="true"/>
+  <xacro:include filename="$(find chassis)/urdf/mecanum.xacro" />
+  <xacro:scan_sensor prefix="scan" use_sim="$(arg use_sim)"/>
+  <xacro:mecanum_drive use_sim="$(arg use_sim)" config_path="${mecanum_config}"/>
   <link
     name="base_link">
@@ -312,51 +316,3 @@
       xyz="0 1 0" />
   </joint>
-  <gazebo reference="FL_Link">
-    <mu1>100.0</mu1>
-    <mu2>100.0</mu2>
-    <kp>100000000.0</kp>
-    <kd>10.0</kd>
-  </gazebo>
-  <gazebo reference="FR_Link">
-    <mu1>100.0</mu1>
-    <mu2>100.0</mu2>
-    <kp>100000000.0</kp>
-    <kd>10.0</kd>
-  </gazebo>
-  <gazebo reference="BL_Link">
-    <mu1>100.0</mu1>
-    <mu2>100.0</mu2>
-    <kp>100000000.0</kp>
-    <kd>10.0</kd>
-  </gazebo>
-  <gazebo reference="BR_Link">
-    <mu1>100.0</mu1>
-    <mu2>100.0</mu2>
-    <kp>100000000.0</kp>
-    <kd>10.0</kd>
-  </gazebo>
-  <gazebo>
-    <plugin name="my_mecanum_plugin" filename="libmecanum_drive_plugin.so">
-      <fl_joint>FL_Joint</fl_joint>
-      <fr_joint>FR_Joint</fr_joint>
-      <bl_joint>BL_Joint</bl_joint>
-      <br_joint>BR_Joint</br_joint>
-      <wheel_radius>0.0375</wheel_radius>
-      <wheel_base>0.1550</wheel_base>
-      <track_width>0.4166</track_width>
-    </plugin>
-  </gazebo>
-  <gazebo>
-    <plugin name="joint_state_publisher" filename="libgazebo_ros_joint_state_publisher.so">
-      <ros>
-        <remapping>~/out:=joint_states</remapping>
-      </ros>
-      <update_rate>50</update_rate>
-      <joint_name>FL_Joint</joint_name>
-      <joint_name>FR_Joint</joint_name>
-      <joint_name>BL_Joint</joint_name>
-      <joint_name>BR_Joint</joint_name>
-    </plugin>
-  </gazebo>
-  <xacro:scan_sensor prefix="scan" use_sim="$(arg use_sim)"/>
 </robot>

File: chassis/urdf/chassis.xacro (robot description, xacro)
@@ -5,6 +5,10 @@
 <robot name="chassis" xmlns:xacro="http://www.ros.org/wiki/xacro">
   <!-- ========== 仿真/实物切换参数 ========== -->
+  <xacro:arg name="use_sim" default="true"/>
+  <xacro:property name="mecanum_config" value="$(find chassis)/config/robot_config.yaml" />
   <xacro:include filename="$(find chassis)/urdf/scan_sensor.xacro" />
-  <xacro:arg name="use_sim" default="true"/>
+  <xacro:include filename="$(find chassis)/urdf/mecanum.xacro" />
+  <xacro:scan_sensor prefix="scan" use_sim="$(arg use_sim)"/>
+  <xacro:mecanum_drive use_sim="$(arg use_sim)" config_path="${mecanum_config}"/>
   <link
     name="base_link">
@@ -312,4 +316,3 @@
       xyz="0 1 0" />
   </joint>
-  <xacro:scan_sensor prefix="scan" use_sim="$(arg use_sim)"/>
 </robot>

File: chassis/urdf/mecanum.xacro (robot description, xacro)
@@ -1,29 +1,17 @@
 <?xml version="1.0"?>
 <robot xmlns:xacro="http://www.ros.org/wiki/xacro">
-  <xacro:macro name="mecanum_drive" params="use_sim:=true">
+  <xacro:macro name="mecanum_drive" params="use_sim:=true config_path:=''">
     <xacro:if value="${use_sim}">
       <gazebo>
-        <plugin name="mecanum_drive" filename="libgazebo_ros_mecanum_drive.so">
-          <ros>
-            <remapping>cmd_vel:=cmd_vel</remapping>
-          </ros>
-          <left_front_joint>FL_Joint</left_front_joint>
-          <right_front_joint>FR_Joint</right_front_joint>
-          <left_rear_joint>BL_Joint</left_rear_joint>
-          <right_rear_joint>BR_Joint</right_rear_joint>
-          <wheel_radius>0.0375</wheel_radius>
-          <wheel_separation>0.4166</wheel_separation>
-          <wheel_base>0.1550</wheel_base>
-          <robot_base_frame>base_link</robot_base_frame>
-          <odometry_frame>odom</odometry_frame>
-          <publish_wheel_tf>false</publish_wheel_tf>
-          <publish_odometry>true</publish_odometry>
-          <publish_odom_tf>true</publish_odom_tf>
+        <plugin name="my_mecanum_plugin" filename="libmecanum_drive_plugin.so">
+          <config_file>${config_path}</config_file>
         </plugin>
+      </gazebo>
+      <gazebo>
         <plugin name="joint_state_publisher" filename="libgazebo_ros_joint_state_publisher.so">
           <ros>
             <remapping>~/out:=joint_states</remapping>
           </ros>
-          <update_rate>30</update_rate>
+          <update_rate>50</update_rate>
           <joint_name>FL_Joint</joint_name>
           <joint_name>FR_Joint</joint_name>

Commit message: Refactor code structure for improved readability and maintainability

File: chassis/install/chassis/share/chassis/urdf/chassis.xacro (robot description, xacro)
@@ -15,15 +15,15 @@
     <inertial>
       <origin
-        xyz="-0.0677499107956596 4.3724418912483E-05 0.0683926250538354"
-        rpy="0 0 0" />
-      <mass
-        value="3.22393142364253" />
-      <inertia
-        ixx="0.0187770652552285"
-        ixy="-6.94989088987062E-08"
-        ixz="-3.69535574562707E-08"
-        iyy="0.02048392582904"
-        iyz="3.35166257416731E-11"
-        izz="0.0375088689683629" />
+        xyz="-0.0677499107745156 4.37244521654945E-05 0.068392625026961"
+        rpy="0 0 0" />
+      <mass
+        value="3.22393142434326" />
+      <inertia
+        ixx="0.0187770652552215"
+        ixy="-6.94990243935453E-08"
+        ixz="-3.69534006071456E-08"
+        iyy="0.0204839258293414"
+        iyz="3.35294125226089E-11"
+        izz="0.0375088689684911" />
     </inertial>
     <visual>
@@ -55,15 +55,15 @@
     <inertial>
       <origin
-        xyz="-0.0025063 4.5658E-06 0.0060826"
-        rpy="0 0 0" />
-      <mass
-        value="0.037431" />
-      <inertia
-        ixx="2.8048E-05"
-        ixy="-2.199E-09"
-        ixz="-1.0712E-06"
-        iyy="3.3616E-05"
-        iyz="-6.8397E-10"
-        izz="4.5085E-05" />
+        xyz="-0.00250631530381856 4.56584855934583E-06 0.00608264669060467"
+        rpy="0 0 0" />
+      <mass
+        value="0.037430735750063" />
+      <inertia
+        ixx="2.80476493089794E-05"
+        ixy="-2.19899695273233E-09"
+        ixz="-1.07121854785533E-06"
+        iyy="3.36164872296788E-05"
+        iyz="-6.83968852525854E-10"
+        izz="4.50845442757729E-05" />
     </inertial>
     <visual>
@@ -78,5 +78,5 @@
         name="">
         <color
-          rgba="0.37647 0.37647 0.37647 1" />
+          rgba="0.376470588235294 0.376470588235294 0.376470588235294 1" />
       </material>
     </visual>
@@ -95,5 +95,5 @@
     type="fixed">
     <origin
-      xyz="0.176999549642127 0 0.0500745386389849"
+      xyz="0.177 0 0.050075"
       rpy="0 0 0" />
     <parent
@@ -108,15 +108,15 @@
     <inertial>
       <origin
-        xyz="-2.268E-05 -0.017766 -3.3245E-05"
-        rpy="0 0 0" />
-      <mass
-        value="0.057098" />
-      <inertia
-        ixx="2.1034E-05"
-        ixy="5.4288E-09"
-        ixz="9.6894E-09"
-        iyy="3.3961E-05"
-        iyz="7.9775E-09"
-        izz="2.1037E-05" />
+        xyz="-1.51557746422698E-05 -0.0177688130626312 3.72943823484378E-05"
+        rpy="0 0 0" />
+      <mass
+        value="0.0570991876952128" />
+      <inertia
+        ixx="2.10306084770148E-05"
+        ixy="-3.63266955109737E-09"
+        ixz="-8.13885817974439E-09"
+        iyy="3.39619809949368E-05"
+        iyz="8.94029294404181E-09"
+        izz="2.1041688188619E-05" />
     </inertial>
     <visual>
@@ -131,5 +131,5 @@
         name="">
         <color
-          rgba="0.79216 0.81961 0.93333 1" />
+          rgba="0.792156862745098 0.819607843137255 0.933333333333333 1" />
       </material>
     </visual>
@@ -148,5 +148,5 @@
     type="continuous">
     <origin
-      xyz="0.0119843681259687 0.207999999999991 -0.0618699701855335"
+      xyz="0.011984 0.207 -0.06187"
       rpy="0 0 0" />
     <parent
@@ -161,15 +161,15 @@
     <inertial>
       <origin
-        xyz="-2.268E-05 0.017753 -3.3245E-05"
-        rpy="0 0 0" />
-      <mass
-        value="0.057098" />
-      <inertia
-        ixx="2.1034E-05"
-        ixy="5.4288E-09"
-        ixz="9.6894E-09"
-        iyy="3.3961E-05"
-        iyz="7.9775E-09"
-        izz="2.1037E-05" />
+        xyz="3.73138131217893E-05 0.0177656337718318 -1.51714675786438E-05"
+        rpy="0 0 0" />
+      <mass
+        value="0.0570982559843118" />
+      <inertia
+        ixx="2.10412305440831E-05"
+        ixy="-8.94174558072254E-09"
+        ixz="-8.14257477486789E-09"
+        iyy="3.39612560042682E-05"
+        iyz="3.63772364271833E-09"
+        izz="2.10301739676632E-05" />
     </inertial>
     <visual>
@@ -184,5 +184,5 @@
         name="">
         <color
-          rgba="0.79216 0.81961 0.93333 1" />
+          rgba="0.792156862745098 0.819607843137255 0.933333333333333 1" />
       </material>
     </visual>
@@ -201,5 +201,5 @@
     type="continuous">
     <origin
-      xyz="0.0119843681259713 -0.207999999999984 -0.061869970185527"
+      xyz="0.011984 -0.206 -0.06187"
       rpy="0 0 0" />
     <parent
@@ -214,15 +214,15 @@
     <inertial>
       <origin
-        xyz="-2.268E-05 -0.017766 -3.3245E-05"
-        rpy="0 0 0" />
-      <mass
-        value="0.057098" />
-      <inertia
-        ixx="2.1034E-05"
-        ixy="5.4288E-09"
-        ixz="9.6894E-09"
-        iyy="3.3961E-05"
-        iyz="7.9775E-09"
-        izz="2.1037E-05" />
+        xyz="3.7313813121137E-05 -0.0177656337718317 1.51714675792752E-05"
+        rpy="0 0 0" />
+      <mass
+        value="0.0570982559843118" />
+      <inertia
+        ixx="2.10412305440832E-05"
+        ixy="8.94174558053171E-09"
+        ixz="8.14257477489918E-09"
+        iyy="3.39612560042682E-05"
+        iyz="3.63772364284194E-09"
+        izz="2.10301739676631E-05" />
     </inertial>
     <visual>
@@ -237,5 +237,5 @@
         name="">
         <color
-          rgba="0.79216 0.81961 0.93333 1" />
+          rgba="0.792156862745098 0.819607843137255 0.933333333333333 1" />
       </material>
     </visual>
@@ -254,5 +254,5 @@
     type="continuous">
     <origin
-      xyz="-0.14301563187372 0.207999999999992 -0.0618702809722271"
+      xyz="-0.14302 0.206 -0.06187"
       rpy="0 0 0" />
     <parent
@@ -267,15 +267,15 @@
     <inertial>
       <origin
-        xyz="-2.268E-05 0.017753 -3.3245E-05"
-        rpy="0 0 0" />
-      <mass
-        value="0.057098" />
-      <inertia
-        ixx="2.1034E-05"
-        ixy="5.4288E-09"
-        ixz="9.6894E-09"
-        iyy="3.3961E-05"
-        iyz="7.9775E-09"
-        izz="2.1037E-05" />
+        xyz="1.51557746424433E-05 0.017768813062631 3.72943823481672E-05"
+        rpy="0 0 0" />
+      <mass
+        value="0.0570991876952133" />
+      <inertia
+        ixx="2.10306084770149E-05"
+        ixy="-3.63266955067876E-09"
+        ixz="8.13885817975177E-09"
+        iyy="3.3961980994937E-05"
+        iyz="-8.9402929444889E-09"
+        izz="2.10416881886191E-05" />
     </inertial>
     <visual>
@@ -290,5 +290,5 @@
         name="">
         <color
-          rgba="0.79216 0.81961 0.93333 1" />
+          rgba="0.792156862745098 0.819607843137255 0.933333333333333 1" />
       </material>
     </visual>
@@ -307,5 +307,5 @@
     type="continuous">
     <origin
-      xyz="-0.143015631873717 -0.207999999999986 -0.0618702809722206"
+      xyz="-0.14302 -0.207 -0.06187"
       rpy="0 0 0" />
     <parent

File: chassis/urdf/chassis.urdf (robot description, URDF)
Before this commit: robot chassis, 6 links, 5 joints
Links:
- link BL_Link: mass 0.057098 -> 0.0570982559843118
- link BR_Link: mass 0.057098 -> 0.0570991876952133
- link FL_Link: mass 0.057098 -> 0.0570991876952128
- link FR_Link: mass 0.057098 -> 0.0570982559843118
- link base_link: mass 3.22393142364253 -> 3.22393142434326
- link scan_Link: mass 0.037431 -> 0.037430735750063
Joints:
- joint BL_Joint: origin xyz=-0.14301563187372 0.207999999999992 -0.0618702809722271 rpy=0 0 0 -> xyz=-0.14302 0.206 -0.06187 rpy=0 0 0
- joint BR_Joint: origin xyz=-0.143015631873717 -0.207999999999986 -0.0618702809722206 rpy=0 0 0 -> xyz=-0.14302 -0.207 -0.06187 rpy=0 0 0
- joint FL_Joint: origin xyz=0.0119843681259687 0.207999999999991 -0.0618699701855335 rpy=0 0 0 -> xyz=0.011984 0.207 -0.06187 rpy=0 0 0
- joint FR_Joint: origin xyz=0.0119843681259713 -0.207999999999984 -0.061869970185527 rpy=0 0 0 -> xyz=0.011984 -0.206 -0.06187 rpy=0 0 0
- joint scan_Joint: origin xyz=0.176999549642127 0 0.0500745386389849 rpy=0 0 0 -> xyz=0.177 0 0.050075 rpy=0 0 0

File: chassis/urdf/chassis.xacro (robot description, xacro)
@@ -5,8 +5,22 @@
 <robot name="chassis" xmlns:xacro="http://www.ros.org/wiki/xacro">
   <!-- ========== 仿真/实物切换参数 ========== -->
+  <!-- 接收从 launch 传入的物理参数（需与 launch 中 xacro 参数名一致） -->
+  <xacro:arg name="wheel_mu1" default="0.8"/>
+  <xacro:arg name="wheel_mu2" default="0.6"/>
+  <xacro:arg name="wheel_kp" default="100000.0"/>
+  <xacro:arg name="wheel_kd" default="10.0"/>
   <xacro:arg name="use_sim" default="true"/>
   <xacro:property name="mecanum_config" value="$(find chassis)/config/robot_config.yaml" />
   <xacro:include filename="$(find chassis)/urdf/scan_sensor.xacro" />
   <xacro:include filename="$(find chassis)/urdf/mecanum.xacro" />
+  <!-- 调用宏，传入物理参数 -->
+  <xacro:mecanum_drive
+      use_sim="$(arg use_sim)"
+      config_path="$(find chassis)/config/robot_config.yaml"
+      wheel_mu1="$(arg wheel_mu1)"
+      wheel_mu2="$(arg wheel_mu2)"
+      wheel_kp="$(arg wheel_kp)"
+      wheel_kd="$(arg wheel_kd)"
+  />
   <xacro:scan_sensor prefix="scan" use_sim="$(arg use_sim)"/>
   <xacro:mecanum_drive use_sim="$(arg use_sim)" config_path="${mecanum_config}"/>
@@ -15,15 +29,15 @@
     <inertial>
       <origin
-        xyz="-0.0677499107956596 4.3724418912483E-05 0.0683926250538354"
-        rpy="0 0 0" />
-      <mass
-        value="3.22393142364253" />
-      <inertia
-        ixx="0.0187770652552285"
-        ixy="-6.94989088987062E-08"
-        ixz="-3.69535574562707E-08"
-        iyy="0.02048392582904"
-        iyz="3.35166257416731E-11"
-        izz="0.0375088689683629" />
+        xyz="-0.0677499107745156 4.37244521654945E-05 0.068392625026961"
+        rpy="0 0 0" />
+      <mass
+        value="3.22393142434326" />
+      <inertia
+        ixx="0.0187770652552215"
+        ixy="-6.94990243935453E-08"
+        ixz="-3.69534006071456E-08"
+        iyy="0.0204839258293414"
+        iyz="3.35294125226089E-11"
+        izz="0.0375088689684911" />
     </inertial>
     <visual>
@@ -55,15 +69,15 @@
     <inertial>
       <origin
-        xyz="-0.0025063 4.5658E-06 0.0060826"
-        rpy="0 0 0" />
-      <mass
-        value="0.037431" />
-      <inertia
-        ixx="2.8048E-05"
-        ixy="-2.199E-09"
-        ixz="-1.0712E-06"
-        iyy="3.3616E-05"
-        iyz="-6.8397E-10"
-        izz="4.5085E-05" />
+        xyz="-0.00250631530381856 4.56584855934583E-06 0.00608264669060467"
+        rpy="0 0 0" />
+      <mass
+        value="0.037430735750063" />
+      <inertia
+        ixx="2.80476493089794E-05"
+        ixy="-2.19899695273233E-09"
+        ixz="-1.07121854785533E-06"
+        iyy="3.36164872296788E-05"
+        iyz="-6.83968852525854E-10"
+        izz="4.50845442757729E-05" />
     </inertial>
     <visual>
@@ -78,5 +92,5 @@
         name="">
         <color
-          rgba="0.37647 0.37647 0.37647 1" />
+          rgba="0.376470588235294 0.376470588235294 0.376470588235294 1" />
       </material>
     </visual>
@@ -95,5 +109,5 @@
     type="fixed">
     <origin
-      xyz="0.176999549642127 0 0.0500745386389849"
+      xyz="0.177 0 0.050075"
       rpy="0 0 0" />
     <parent
@@ -108,15 +122,15 @@
     <inertial>
       <origin
-        xyz="-2.268E-05 -0.017766 -3.3245E-05"
-        rpy="0 0 0" />
-      <mass
-        value="0.057098" />
-      <inertia
-        ixx="2.1034E-05"
-        ixy="5.4288E-09"
-        ixz="9.6894E-09"
-        iyy="3.3961E-05"
-        iyz="7.9775E-09"
-        izz="2.1037E-05" />
+        xyz="-1.51557746422698E-05 -0.0177688130626312 3.72943823484378E-05"
+        rpy="0 0 0" />
+      <mass
+        value="0.0570991876952128" />
+      <inertia
+        ixx="2.10306084770148E-05"
+        ixy="-3.63266955109737E-09"
+        ixz="-8.13885817974439E-09"
+        iyy="3.39619809949368E-05"
+        iyz="8.94029294404181E-09"
+        izz="2.1041688188619E-05" />
     </inertial>
     <visual>
@@ -131,5 +145,5 @@
         name="">
         <color
-          rgba="0.79216 0.81961 0.93333 1" />
+          rgba="0.792156862745098 0.819607843137255 0.933333333333333 1" />
       </material>
     </visual>
@@ -148,5 +162,5 @@
     type="continuous">
     <origin
-      xyz="0.0119843681259687 0.207999999999991 -0.0618699701855335"
+      xyz="0.011984 0.207 -0.06187"
       rpy="0 0 0" />
     <parent
@@ -161,15 +175,15 @@
     <inertial>
       <origin
-        xyz="-2.268E-05 0.017753 -3.3245E-05"
-        rpy="0 0 0" />
-      <mass
-        value="0.057098" />
-      <inertia
-        ixx="2.1034E-05"
-        ixy="5.4288E-09"
-        ixz="9.6894E-09"
-        iyy="3.3961E-05"
-        iyz="7.9775E-09"
-        izz="2.1037E-05" />
+        xyz="3.73138131217893E-05 0.0177656337718318 -1.51714675786438E-05"
+        rpy="0 0 0" />
+      <mass
+        value="0.0570982559843118" />
+      <inertia
+        ixx="2.10412305440831E-05"
+        ixy="-8.94174558072254E-09"
+        ixz="-8.14257477486789E-09"
+        iyy="3.39612560042682E-05"
+        iyz="3.63772364271833E-09"
+        izz="2.10301739676632E-05" />
     </inertial>
     <visual>
@@ -184,5 +198,5 @@
         name="">
         <color
-          rgba="0.79216 0.81961 0.93333 1" />
+          rgba="0.792156862745098 0.819607843137255 0.933333333333333 1" />
       </material>
     </visual>
@@ -201,5 +215,5 @@
     type="continuous">
     <origin
-      xyz="0.0119843681259713 -0.207999999999984 -0.061869970185527"
+      xyz="0.011984 -0.206 -0.06187"
       rpy="0 0 0" />
     <parent
@@ -214,15 +228,15 @@
     <inertial>
       <origin
-        xyz="-2.268E-05 -0.017766 -3.3245E-05"
-        rpy="0 0 0" />
-      <mass
-        value="0.057098" />
-      <inertia
-        ixx="2.1034E-05"
-        ixy="5.4288E-09"
-        ixz="9.6894E-09"
-        iyy="3.3961E-05"
-        iyz="7.9775E-09"
-        izz="2.1037E-05" />
+        xyz="3.7313813121137E-05 -0.0177656337718317 1.51714675792752E-05"
+        rpy="0 0 0" />
+      <mass
+        value="0.0570982559843118" />
+      <inertia
+        ixx="2.10412305440832E-05"
+        ixy="8.94174558053171E-09"
+        ixz="8.14257477489918E-09"
+        iyy="3.39612560042682E-05"
+        iyz="3.63772364284194E-09"
+        izz="2.10301739676631E-05" />
     </inertial>
     <visual>
@@ -237,5 +251,5 @@
         name="">
         <color
-          rgba="0.79216 0.81961 0.93333 1" />
+          rgba="0.792156862745098 0.819607843137255 0.933333333333333 1" />
       </material>
     </visual>
@@ -254,5 +268,5 @@
     type="continuous">
     <origin
-      xyz="-0.14301563187372 0.207999999999992 -0.0618702809722271"
+      xyz="-0.14302 0.206 -0.06187"
       rpy="0 0 0" />
     <parent
@@ -267,15 +281,15 @@
     <inertial>
       <origin
-        xyz="-2.268E-05 0.017753 -3.3245E-05"
-        rpy="0 0 0" />
-      <mass
-        value="0.057098" />
-      <inertia
-        ixx="2.1034E-05"
-        ixy="5.4288E-09"
-        ixz="9.6894E-09"
-        iyy="3.3961E-05"
-        iyz="7.9775E-09"
-        izz="2.1037E-05" />
+        xyz="1.51557746424433E-05 0.017768813062631 3.72943823481672E-05"
+        rpy="0 0 0" />
+      <mass
+        value="0.0570991876952133" />
+      <inertia
+        ixx="2.10306084770149E-05"
+        ixy="-3.63266955067876E-09"
+        ixz="8.13885817975177E-09"
+        iyy="3.3961980994937E-05"
+        iyz="-8.9402929444889E-09"
+        izz="2.10416881886191E-05" />
     </inertial>
     <visual>
@@ -290,5 +304,5 @@
         name="">
         <color
-          rgba="0.79216 0.81961 0.93333 1" />
+          rgba="0.792156862745098 0.819607843137255 0.933333333333333 1" />
       </material>
     </visual>
@@ -307,5 +321,5 @@
     type="continuous">
     <origin
-      xyz="-0.143015631873717 -0.207999999999986 -0.0618702809722206"
+      xyz="-0.14302 -0.207 -0.06187"
       rpy="0 0 0" />
     <parent

File: chassis/urdf/mecanum.xacro (robot description, xacro)
@@ -1,6 +1,8 @@
 <?xml version="1.0"?>
 <robot xmlns:xacro="http://www.ros.org/wiki/xacro">
-  <xacro:macro name="mecanum_drive" params="use_sim:=true config_path:=''">
+  <xacro:macro name="mecanum_drive" params="use_sim:=true config_path:=''
+               wheel_mu1:=0.8 wheel_mu2:=0.6 wheel_kp:=100000.0 wheel_kd:=10.0">
     <xacro:if value="${use_sim}">
+      <!-- 自定义麦轮驱动插件 -->
       <gazebo>
         <plugin name="my_mecanum_plugin" filename="libmecanum_drive_plugin.so">
@@ -8,4 +10,5 @@
         </plugin>
       </gazebo>
+      <!-- 关节状态发布插件 -->
       <gazebo>
         <plugin name="joint_state_publisher" filename="libgazebo_ros_joint_state_publisher.so">
@@ -20,4 +23,29 @@
         </plugin>
       </gazebo>
+      <!-- 轮子物理属性（统一配置） -->
+      <gazebo reference="FL_Link">
+        <mu1>${wheel_mu1}</mu1>
+        <mu2>${wheel_mu2}</mu2>
+        <kp>${wheel_kp}</kp>
+        <kd>${wheel_kd}</kd>
+      </gazebo>
+      <gazebo reference="FR_Link">
+        <mu1>${wheel_mu1}</mu1>
+        <mu2>${wheel_mu2}</mu2>
+        <kp>${wheel_kp}</kp>
+        <kd>${wheel_kd}</kd>
+      </gazebo>
+      <gazebo reference="BL_Link">
+        <mu1>${wheel_mu1}</mu1>
+        <mu2>${wheel_mu2}</mu2>
+        <kp>${wheel_kp}</kp>
+        <kd>${wheel_kd}</kd>
+      </gazebo>
+      <gazebo reference="BR_Link">
+        <mu1>${wheel_mu1}</mu1>
+        <mu2>${wheel_mu2}</mu2>
+        <kp>${wheel_kp}</kp>
+        <kd>${wheel_kd}</kd>
+      </gazebo>
     </xacro:if>
   </xacro:macro>
