Commit message: 缓存

File: src/nav_stack_core/description/minimal_lidar_robot.xacro (robot description, xacro)
@@ -1,4 +1,5 @@
 <?xml version="1.0"?>
 <robot xmlns:xacro="http://www.ros.org/wiki/xacro" name="fusion_robot">
+  <!-- base_link 为底盘刚体参考系 -->
   <!-- IMU 相对 base_link 的安装位置 -->
   <xacro:arg name="imu_x" default="0.00"/>
@@ -8,8 +9,8 @@
   <xacro:arg name="imu_pitch" default="0.0"/>
   <xacro:arg name="imu_yaw" default="0.0"/>
-  <!-- 雷达相对 imu_link 的安装位置 -->
+  <!-- 激光雷达相对 base_link 的安装位置 -->
   <xacro:arg name="laser_x" default="0.10"/>
   <xacro:arg name="laser_y" default="0.00"/>
-  <xacro:arg name="laser_z" default="0.10"/>
+  <xacro:arg name="laser_z" default="0.15"/>
   <xacro:arg name="laser_roll" default="0.0"/>
   <xacro:arg name="laser_pitch" default="0.0"/>
@@ -18,5 +19,5 @@
   <link name="imu_link"/>
   <link name="laser"/>
-  <!-- IMU 挂在 base_link 上 -->
+  <!-- IMU 刚性固定在底盘上 -->
   <joint name="base_to_imu" type="fixed">
     <parent link="base_link"/>
@@ -25,7 +26,7 @@
             rpy="$(arg imu_roll) $(arg imu_pitch) $(arg imu_yaw)"/>
   </joint>
-  <!-- 雷达挂在 imu_link 上，坐标系跟着 imu_link -->
-  <joint name="imu_to_laser" type="fixed">
-    <parent link="imu_link"/>
+  <!-- 激光雷达直接刚性固定在底盘上，不挂在 imu_link 下面 -->
+  <joint name="base_to_laser" type="fixed">
+    <parent link="base_link"/>
     <child link="laser"/>
     <origin xyz="$(arg laser_x) $(arg laser_y) $(arg laser_z)"
