Commit message: temp-v1.0.2

File: src/Diverse/robot2/urdf/robot2.urdf (robot description, URDF)
Before this commit: robot robot2, 7 links, 6 joints
Links:
- removed link cam1_Link
- added link camera_link, mass 0.107926872108232; collision mesh filename=package://robot2/meshes/camera_link.STL; visual mesh filename=package://robot2/meshes/camera_link.STL
Joints:
- joint cam1_Joint: child cam1_Link -> camera_link

File: src/Diverse/robot2/urdf/robot2_expanded.urdf (robot description, URDF)
Before this commit: robot robot2, 7 links, 6 joints
Links:
- removed link cam1_Link
- added link camera_link, mass 0.107926872108232; collision mesh filename=package://robot2/meshes/camera_link.STL; visual mesh filename=package://robot2/meshes/camera_link.STL
Joints:
- joint cam1_Joint: child cam1_Link -> camera_link

Commit message: temp-v1.0.6.2

File: src/Diverse/robot2/urdf/robot2.urdf (robot description, URDF)
Before this commit: robot robot2, 7 links, 6 joints
Links:
- removed link camera_link
- added link Platfrom_Link, mass 0.71015; collision mesh filename=package://robot2/meshes/Platfrom_Link.STL; visual mesh filename=package://robot2/meshes/Platfrom_Link.STL
- added link Rollout_Link, mass 0.72568; collision mesh filename=package://robot2/meshes/Rollout_Link.STL; visual mesh filename=package://robot2/meshes/Rollout_Link.STL
- added link d435-cam-Link, mass 0.107926872108232; collision mesh filename=package://robot2/meshes/d435-cam-Link.STL; visual mesh filename=package://robot2/meshes/d435-cam-Link.STL
- added link oak-cam-Link, mass 0.048473; collision mesh filename=package://robot2/meshes/oak-cam-Link.STL; visual mesh filename=package://robot2/meshes/oak-cam-Link.STL
- link BR-Link: mass 0.524127400676241 -> 0.52413
- link FL-Link: mass 0.524127400675719 -> 0.52413
- link FR-Link: mass 0.524125547602897 -> 0.52413
- link base_link: mass 4.54700799044429 -> 4.5470079909601
Joints:
- removed joint cam1_Joint
- added joint Platfrom_Joint: type prismatic, parent base_link, child Platfrom_Link, origin xyz=-0.000499492705473831 0.0494030997391482 0.14563170765098 rpy=0 0 0, axis 0 0 1, limit lower=0 upper=0 effort=0 velocity=0
- added joint Rollout_Joint: type prismatic, parent Platfrom_Link, child Rollout_Link, origin xyz=0 -0.102913366310849 0.0760000000001064 rpy=0 0 0, axis 0 -1 0, limit lower=0 upper=0 effort=0 velocity=0
- added joint d435-cam-Joint: type fixed, parent base_link, child d435-cam-Link, origin xyz=0.286567199500283 0.0664321363029682 0.40695175281066 rpy=0 0.436332312998575 0, axis 0 0 0
- added joint oak-cam-Joint: type fixed, parent Rollout_Link, child oak-cam-Link, origin xyz=0 0.145219305523008 0.113498999999999 rpy=0 0 -1.57079632679489, axis 0 0 0

Commit message: temp-v1.0.6.3

File: src/Diverse/robot2/urdf/robot2.urdf (robot description, URDF)
Before this commit: robot robot2, 10 links, 9 joints
Links:
- added link camera_link
Joints:
- added joint d435_camera_link_joint: type fixed, parent d435-cam-Link, child camera_link, origin xyz=0 0 0 rpy=0 0 0
